File: fpga-bank-16.kicad_sch (KiCad schematic)
At the start: 3 parts, among them U4 XC7K160T-FFG676, Y3 Oscillator_100MHz_ASFL1

Commit message: [#65754] Rename project
Other:
- title: SO-DIMM DDR5 Tester -> RDIMM DDR5 Tester
Changed lines of the file:
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@@
   (paper "A3")
   (title_block
-    (title "SO-DIMM DDR5 Tester")
-    (date "2024-04-23")
-    (rev "1.2.0")
+    (title "RDIMM DDR5 Tester")
+    (date "2024-09-26")
+    (rev "2.0.0")
     (comment 1 "www.antmicro.com")
     (comment 2 "Antmicro Ltd")
@@
     (pin "1")
     (instances
-      (project "rdimm-ddr5-tester-ultrascale-plus"
+      (project "data-center-rdimm-ddr5-tester"
         (path "/1faa6543-e26a-4449-8bac-ee14b9f19e5f/c1ddaa09-f59e-4e22-abc1-585fde8776d6"
           (reference "#PWR0265") (unit 1)
@@
     (pin "2")
     (instances
-      (project "rdimm-ddr5-tester-ultrascale-plus"
+      (project "data-center-rdimm-ddr5-tester"
         (path "/1faa6543-e26a-4449-8bac-ee14b9f19e5f/c1ddaa09-f59e-4e22-abc1-585fde8776d6"
           (reference "C164") (unit 1)
@@
     (pin "4")
     (instances
-      (project "rdimm-ddr5-tester-ultrascale-plus"
+      (project "data-center-rdimm-ddr5-tester"
         (path "/1faa6543-e26a-4449-8bac-ee14b9f19e5f/c1ddaa09-f59e-4e22-abc1-585fde8776d6"
           (reference "Y3") (unit 1)
@@
     (pin "T6")
     (instances
-      (project "rdimm-ddr5-tester-ultrascale-plus"
+      (project "data-center-rdimm-ddr5-tester"
         (path "/1faa6543-e26a-4449-8bac-ee14b9f19e5f/c1ddaa09-f59e-4e22-abc1-585fde8776d6"
           (reference "U4") (unit 5)
@@
     (pin "1")
     (instances
-      (project "rdimm-ddr5-tester-ultrascale-plus"
+      (project "data-center-rdimm-ddr5-tester"
         (path "/1faa6543-e26a-4449-8bac-ee14b9f19e5f/c1ddaa09-f59e-4e22-abc1-585fde8776d6"
           (reference "#PWR0263") (unit 1)
@@
     (pin "1")
     (instances
-      (project "rdimm-ddr5-tester-ultrascale-plus"
+      (project "data-center-rdimm-ddr5-tester"
         (path "/1faa6543-e26a-4449-8bac-ee14b9f19e5f/c1ddaa09-f59e-4e22-abc1-585fde8776d6"
           (reference "#PWR0264") (unit 1)
@@
     (pin "1")
     (instances
-      (project "rdimm-ddr5-tester-ultrascale-plus"
+      (project "data-center-rdimm-ddr5-tester"
         (path "/1faa6543-e26a-4449-8bac-ee14b9f19e5f/c1ddaa09-f59e-4e22-abc1-585fde8776d6"
           (reference "#PWR0262") (unit 1)
