File: fpga-banks-32-34.kicad_sch (KiCad schematic)
At the start: 9 parts, among them U4 XC7K160T-FFG676

Commit message: [#66311] Add XCAU25P. Reconnect configuration bank 0
Parts:
- added U34: XCAU25P-2FFVB676I, antmicro-footprints:BGA-676_27x27mm_Layout26x26_P1x1mm_FFVB676, symbol antmicroFPGAChips:XCAU25P-2FFVB676I
Connections:
- new net: U34.AC15 (VCCO_84), U34.Y14 (VCCO_84)
- new net: U34.AA21 (VCCO_64), U34.AB18 (VCCO_64), U34.AD22 (VCCO_64)
- new net: U34.E9 (VCCO_86), U34.H10 (VCCO_86)
- new net: U34.E24 (VCCO_66), U34.H25 (VCCO_66), U34.J22 (VCCO_66)
- new net: U34.E14 (VCCO_87), U34.H15 (VCCO_87)
- new net: U34.C20 (VCCO_67), U34.D17 (VCCO_67), U34.G18 (VCCO_67)
- new net: U34.P22 (VCCO_65), U34.U23 (VCCO_65), U34.Y24 (VCCO_65)

Commit message: [#65754] Rename project
Parts:
- removed unit 6 of U34
- removed unit 7 of U34
- removed unit 8 of U34
Connections:
- net +1V1: now also U34.AA21 (VCCO_64), U34.AB18 (VCCO_64), U34.AD22 (VCCO_64), U34.E24 (VCCO_66), U34.H25 (VCCO_66), U34.J22 (VCCO_66), U34.P22 (VCCO_65), U34.U23 (VCCO_65), U34.Y24 (VCCO_65)
Other:
- title: SO-DIMM DDR5 Tester -> RDIMM DDR5 Tester
