File: fpga-bank-13-15.kicad_sch (KiCad schematic)
At the start: 3 parts, among them U4 XC7K160T-FFG676

Commit message: [#65754] Rename project
Other:
- title: SO-DIMM DDR5 Tester -> RDIMM DDR5 Tester
Changed lines of the file:
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@@
   (paper "A3")
   (title_block
-    (title "SO-DIMM DDR5 Tester")
-    (date "2024-04-23")
-    (rev "1.2.0")
+    (title "RDIMM DDR5 Tester")
+    (date "2024-09-26")
+    (rev "2.0.0")
     (comment 1 "www.antmicro.com")
     (comment 2 "Antmicro Ltd")
@@
     (pin "T6")
     (instances
-      (project "rdimm-ddr5-tester-ultrascale-plus"
+      (project "data-center-rdimm-ddr5-tester"
         (path "/1faa6543-e26a-4449-8bac-ee14b9f19e5f/e240eeea-be8a-4736-b415-db6627c3e732"
           (reference "U4") (unit 4)
@@
     (pin "2")
     (instances
-      (project "rdimm-ddr5-tester-ultrascale-plus"
+      (project "data-center-rdimm-ddr5-tester"
         (path "/1faa6543-e26a-4449-8bac-ee14b9f19e5f/e240eeea-be8a-4736-b415-db6627c3e732"
           (reference "R96") (unit 1)
@@
     (pin "1")
     (instances
-      (project "rdimm-ddr5-tester-ultrascale-plus"
+      (project "data-center-rdimm-ddr5-tester"
         (path "/1faa6543-e26a-4449-8bac-ee14b9f19e5f/e240eeea-be8a-4736-b415-db6627c3e732"
           (reference "#FLG0108") (unit 1)
@@
     (pin "1")
     (instances
-      (project "rdimm-ddr5-tester-ultrascale-plus"
+      (project "data-center-rdimm-ddr5-tester"
         (path "/1faa6543-e26a-4449-8bac-ee14b9f19e5f/e240eeea-be8a-4736-b415-db6627c3e732"
           (reference "#PWR0236") (unit 1)
@@
     (pin "2")
     (instances
-      (project "rdimm-ddr5-tester-ultrascale-plus"
+      (project "data-center-rdimm-ddr5-tester"
         (path "/1faa6543-e26a-4449-8bac-ee14b9f19e5f/e240eeea-be8a-4736-b415-db6627c3e732"
           (reference "R97") (unit 1)
@@
     (pin "T6")
     (instances
-      (project "rdimm-ddr5-tester-ultrascale-plus"
+      (project "data-center-rdimm-ddr5-tester"
         (path "/1faa6543-e26a-4449-8bac-ee14b9f19e5f/e240eeea-be8a-4736-b415-db6627c3e732"
           (reference "U4") (unit 2)
@@
     (pin "1")
     (instances
-      (project "rdimm-ddr5-tester-ultrascale-plus"
+      (project "data-center-rdimm-ddr5-tester"
         (path "/1faa6543-e26a-4449-8bac-ee14b9f19e5f/e240eeea-be8a-4736-b415-db6627c3e732"
           (reference "#FLG0109") (unit 1)
@@
     (pin "1")
     (instances
-      (project "rdimm-ddr5-tester-ultrascale-plus"
+      (project "data-center-rdimm-ddr5-tester"
         (path "/1faa6543-e26a-4449-8bac-ee14b9f19e5f/e240eeea-be8a-4736-b415-db6627c3e732"
           (reference "#PWR0238") (unit 1)
