File: i2c.kicad_sch (KiCad schematic)
At the start: 41 parts, among them J12 JST_SH_1x4_BM04B-SRSS-TB-LF-SN, Q22 NX3008NBKW, Q24 NX3008NBKW, U23 TS5A3359_VSSOP, U24 TS5A3359_VSSOP, U33 TPD4E05U06QDQARQ1, U45 PCA9517ADP, U49 TCA39306_VSSOP

Commit message: [#68016] Update I3C circuit
Parts:
- removed Q22, Q24: NX3008NBKW, antmicro-footprints:SOT-323, symbol antmicroTransistorsFETsMOSFETsSingle:NX3008NBKW
- removed R235: R_200k_0402, antmicro-footprints:R_0402_1005Metric, symbol antmicroResistors0402:R_200k_0402
- removed R87: R_47k_0402, antmicro-footprints:R_0402_1005Metric, symbol antmicroResistors0402:R_47k_0402
- added Q21, Q23: BSS84AKW, antmicro-footprints:SOT-323, symbol antmicroTransistorsFETsMOSFETsSingle:BSS84AKW
- added R222: R_0R_0402, antmicro-footprints:R_0402_1005Metric, symbol antmicroResistors0402:R_0R_0402
- added R223: R_47k_0402, antmicro-footprints:R_0402_1005Metric, symbol antmicroResistors0402:R_47k_0402
- added R75: R_200k_0402, antmicro-footprints:R_0402_1005Metric, symbol antmicroResistors0402:R_200k_0402
- R96: now in the parts list
Connections:
- net +1V8: no longer C320.1, U49.2 (Vref1)
- net +3V3: now also Q21.2 (S), R222.2, R223.2, R75.2; no longer C325.2, J12.2
- net FPGA_I3C.SCL: now also R97.1, U49.6 (SCL2); no longer R231.1, U49.4 (SDA1)
- net FPGA_I3C.SDA: now also R231.1, U49.5 (SDA2); no longer R97.1, U49.3 (SCL1)
- net GND: no longer R232.1
- net I3C_EXT.SCL: now also J12.3, R241.1, U49.3 (SCL1); no longer J12.4, R243.1, U49.5 (SDA2)
- net I3C_EXT.SDA: now also J12.4, R243.1, U49.4 (SDA1); no longer J12.3, R241.1, U49.6 (SCL2)
- net ~{FPGA_I3C_EXT_PU}: now also Q21.1 (G), R223.1
- net ~{I3C_EXT_PU}: now also R232.1, Q23.1 (G); no longer R232.2
- net at C324.2, R241.2, R243.2: now also Q23.3 (D)
- net at U49.7 (Vref2), U49.8 (EN): now also C320.1, R75.1; no longer C322.1
- net at R15.1, R96.1: now also C322.1, R232.2, U49.2 (Vref1), Q23.2 (S)
- net at C318.2, R231.2, R97.2: now also Q21.3 (D)
- new net: C325.2, J12.2, R222.1
Other:
- moved on the sheet: C318, C324, C325, R15, R231, R232, R241, R243, R97
