File: i2c.kicad_sch (KiCad schematic)
At the start: 43 parts, among them J12 JST_SH_1x4_BM04B-SRSS-TB-LF-SN, Q22 BSS84AKW, Q24 BSS84AKW, U23 TS5A3359_VSSOP, U24 TS5A3359_VSSOP, U33 TPD4E05U06QDQARQ1, U45 PCA9517ADP, U49 TCA39306_VSSOP

Commit message: Correct company name in project files
Other:
- company: (none) -> Antmicro
Changed lines of the file:
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@@
 		(date "2024-12-20")
 		(rev "2.1.0")
+		(company "Antmicro")
 		(comment 1 "www.antmicro.com")
 		(comment 2 "Antmicro")

Commit message: [#97338] Fix malformed DNP properties
Parts:
- TP7: now left out of the parts list
Changed lines of the file:
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@@
 		(unit 1)
 		(exclude_from_sim no)
-		(in_bom yes)
+		(in_bom no)
 		(on_board yes)
 		(dnp no)
