File: fpga-mgt.kicad_sch (KiCad schematic)
At the start: 50 parts, among them U34 XCAU25P-2FFVB676I, U39 SI5319C-C-GM-ND, Y4 Resonator_114.285MHZ_ABM8

Commit message: [#68016] Solve ERC warrings and errors
Parts:
- R35: footprint antmicro-footprints:R_0402_1005Metric_EIA -> antmicro-footprints:R_0402_1005Metric
Changed lines of the file:
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@@
     )
   )
-  (symbol (lib_name "XCAU25P-2FFVB676I_1") (lib_id "antmicroFPGAChips:XCAU25P-2FFVB676I") (at 278.13 63.5 0) (mirror y) (unit 11)
+  (symbol (lib_id "antmicroFPGAChips:XCAU25P-2FFVB676I") (at 278.13 63.5 0) (mirror y) (unit 11)
     (in_bom yes) (on_board yes) (dnp no)
     (property "Reference" "U34" (at 270.51 53.34 0)
@@
       (effects (font (size 1.27 1.27) (thickness 0.15)) (justify left bottom) hide)
     )
-    (property "Footprint" "antmicro-footprints:R_0402_1005Metric_EIA" (at 285.75 182.88 0)
+    (property "Footprint" "antmicro-footprints:R_0402_1005Metric" (at 285.75 182.88 0)
       (effects (font (size 1.27 1.27) (thickness 0.15)) (justify left bottom) hide)
     )
@@
     )
   )
-  (symbol (lib_name "GND_1") (lib_id "antmicropower:GND") (at 308.61 241.3 0) (unit 1)
+  (symbol (lib_id "antmicropower:GND") (at 308.61 241.3 0) (unit 1)
     (in_bom yes) (on_board yes) (dnp no)
     (property "Reference" "#PWR0425" (at 317.5 243.84 0)
@@
     )
   )
-  (symbol (lib_name "GND_1") (lib_id "antmicropower:GND") (at 300.99 241.3 0) (unit 1)
+  (symbol (lib_id "antmicropower:GND") (at 300.99 241.3 0) (unit 1)
     (in_bom yes) (on_board yes) (dnp no)
     (property "Reference" "#PWR0373" (at 309.88 243.84 0)
@@
     )
   )
-  (symbol (lib_id "antmicroFPGAChips:XCAU25P-2FFVB676I") (at 76.2 154.94 0) (mirror y) (unit 10)
+  (symbol (lib_name "XCAU25P-2FFVB676I_2") (lib_id "antmicroFPGAChips:XCAU25P-2FFVB676I") (at 76.2 154.94 0) (mirror y) (unit 10)
     (in_bom yes) (on_board yes) (dnp no)
     (property "Reference" "U34" (at 68.58 144.145 0)

Commit message: [#68199] Start implementing changes after the PCB review
Parts:
- R35: footprint antmicro-footprints:R_0402_1005Metric -> antmicro-footprints:R_0402_1005Metric_EIA
Changed lines of the file:
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@@
       (effects (font (size 1.27 1.27) (thickness 0.15)) (justify left bottom) hide)
     )
-    (property "Footprint" "antmicro-footprints:R_0402_1005Metric" (at 285.75 182.88 0)
+    (property "Footprint" "antmicro-footprints:R_0402_1005Metric_EIA" (at 285.75 182.88 0)
       (effects (font (size 1.27 1.27) (thickness 0.15)) (justify left bottom) hide)
     )
