File: ddr5-rdimm.kicad_sch (KiCad schematic)
At the start: 34 parts, among them J2 Bus_DDR5_DDR504111002KQ, Q10 BSS138PW, Q11 BSS138PW, Q23 SI7613DN-T1-GE3, Q25 BSS138PW, Q26 BSS138PW, Q27 SI7613DN-T1-GE3, Q9 BSS138PW, SW3 SW_KMR211NGLFS_SMD

Commit message: [#68088] Add heater connector
Parts:
- removed C319, C7: C_4u7_0402, antmicro-footprints:C_0402_1005Metric, symbol antmicroCapacitors0402:C_4u7_0402
- added C319, C7: C_10u_25V_0603, antmicro-footprints:C_0603_1608Metric, symbol antmicroCapacitors0603:C_10u_25V_0603
Connections:
- net GND: now also C319.1, C7.1
- net VIN_BULK: now also C7.2
- net VIN_MGMT: now also C319.2
Changed lines of the file:
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@@
     (effects (font (size 1.27 1.27)) (justify left))
+  )
+  (symbol (lib_id "antmicroCapacitors0603:C_10u_25V_0603") (at 281.94 99.06 90) (unit 1)
+    (in_bom yes) (on_board yes) (dnp no) (fields_autoplaced)
+    (property "Reference" "C7" (at 284.48 95.2436 90)
+      (effects (font (size 1.27 1.27) (thickness 0.15)) (justify right))
+    )
+    (property "Value" "C_10u_25V_0603" (at 292.1 78.74 0)
+      (effects (font (size 1.27 1.27) (thickness 0.15)) (justify left bottom) hide)
+    )
+    (property "Footprint" "antmicro-footprints:C_0603_1608Metric" (at 294.64 78.74 0)
+      (effects (font (size 1.27 1.27) (thickness 0.15)) (justify left bottom) hide)
+    )
+    (property "Datasheet" "https://product.tdk.com/en/search/capacitor/ceramic/mlcc/info?part_no=C1608X5R1E106M080AC" (at 297.18 78.74 0)
+      (effects (font (size 1.27 1.27) (thickness 0.15)) (justify left bottom) hide)
+    )
+    (property "MPN" "C1608X5R1E106M080AC" (at 299.72 78.74 0)
+      (effects (font (size 1.27 1.27) (thickness 0.15)) (justify left bottom) hide)
+    )
+    (property "Manufacturer" "TDK" (at 302.26 78.74 0)
+      (effects (font (size 1.27 1.27) (thickness 0.15)) (justify left bottom) hide)
+    )
+    (property "License" "Apache-2.0" (at 304.8 78.74 0)
+      (effects (font (size 1.27 1.27) (thickness 0.15)) (justify left bottom) hide)
+    )
+    (property "Author" "Antmicro" (at 307.34 78.74 0)
+      (effects (font (size 1.27 1.27) (thickness 0.15)) (justify left bottom) hide)
+    )
+    (property "Val" "10u" (at 284.48 97.7836 90)
+      (effects (font (size 1.27 1.27) (thickness 0.15)) (justify right))
+    )
+    (property "Voltage" "25V" (at 309.88 78.74 0)
+      (effects (font (size 1.27 1.27)) (justify left bottom) hide)
+    )
+    (property "Dielectric" "" (at 312.42 78.74 0)
+      (effects (font (size 1.27 1.27)) (justify left bottom) hide)
+    )
+    (pin "2")
+    (pin "1")
+    (instances
+      (project "data-center-rdimm-ddr5-tester"
+        (path "/1faa6543-e26a-4449-8bac-ee14b9f19e5f/00000000-0000-0000-0000-000061827943"
+          (reference "C7") (unit 1)
+        )
+      )
+    )
   )
   (symbol (lib_id "antmicroResistors0402:R_330R_0402") (at 288.29 161.29 270) (unit 1)
@@
     )
   )
+  (symbol (lib_id "antmicroCapacitors0603:C_10u_25V_0603") (at 281.94 115.57 90) (unit 1)
+    (in_bom yes) (on_board yes) (dnp no) (fields_autoplaced)
+    (property "Reference" "C319" (at 284.48 111.7536 90)
+      (effects (font (size 1.27 1.27) (thickness 0.15)) (justify right))
+    )
+    (property "Value" "C_10u_25V_0603" (at 292.1 95.25 0)
+      (effects (font (size 1.27 1.27) (thickness 0.15)) (justify left bottom) hide)
+    )
+    (property "Footprint" "antmicro-footprints:C_0603_1608Metric" (at 294.64 95.25 0)
+      (effects (font (size 1.27 1.27) (thickness 0.15)) (justify left bottom) hide)
+    )
+    (property "Datasheet" "https://product.tdk.com/en/search/capacitor/ceramic/mlcc/info?part_no=C1608X5R1E106M080AC" (at 297.18 95.25 0)
+      (effects (font (size 1.27 1.27) (thickness 0.15)) (justify left bottom) hide)
+    )
+    (property "MPN" "C1608X5R1E106M080AC" (at 299.72 95.25 0)
+      (effects (font (size 1.27 1.27) (thickness 0.15)) (justify left bottom) hide)
+    )
+    (property "Manufacturer" "TDK" (at 302.26 95.25 0)
+      (effects (font (size 1.27 1.27) (thickness 0.15)) (justify left bottom) hide)
+    )
+    (property "License" "Apache-2.0" (at 304.8 95.25 0)
+      (effects (font (size 1.27 1.27) (thickness 0.15)) (justify left bottom) hide)
+    )
+    (property "Author" "Antmicro" (at 307.34 95.25 0)
+      (effects (font (size 1.27 1.27) (thickness 0.15)) (justify left bottom) hide)
+    )
+    (property "Val" "10u" (at 284.48 114.2936 90)
+      (effects (font (size 1.27 1.27) (thickness 0.15)) (justify right))
+    )
+    (property "Voltage" "25V" (at 309.88 95.25 0)
+      (effects (font (size 1.27 1.27)) (justify left bottom) hide)
+    )
+    (property "Dielectric" "" (at 312.42 95.25 0)
+      (effects (font (size 1.27 1.27)) (justify left bottom) hide)
+    )
+    (pin "2")
+    (pin "1")
+    (instances
+      (project "data-center-rdimm-ddr5-tester"
+        (path "/1faa6543-e26a-4449-8bac-ee14b9f19e5f/00000000-0000-0000-0000-000061827943"
+          (reference "C319") (unit 1)
+        )
+      )
+    )
+  )
   (symbol (lib_id "antmicroTransistorsFETsMOSFETsSingle:BSS138PW") (at 218.44 52.07 0) (unit 1)
     (in_bom yes) (on_board yes) (dnp no)
@@
         (path "/1faa6543-e26a-4449-8bac-ee14b9f19e5f/00000000-0000-0000-0000-000061827943"
           (reference "C127") (unit 1)
-        )
-      )
-    )
-  )
-  (symbol (lib_id "antmicroCapacitors0402:C_4u7_0402") (at 281.94 93.98 270) (unit 1)
-    (in_bom yes) (on_board yes) (dnp no) (fields_autoplaced)
-    (property "Reference" "C7" (at 284.48 95.2563 90)
-      (effects (font (size 1.27 1.27)) (justify left))
-    )
-    (property "Value" "C_4u7_0402" (at 271.78 114.3 0)
-      (effects (font (size 1.27 1.27) (thickness 0.15)) (justify left bottom) hide)
-    )
-    (property "Footprint" "antmicro-footprints:C_0402_1005Metric" (at 269.24 114.3 0)
-      (effects (font (size 1.27 1.27) (thickness 0.15)) (justify left bottom) hide)
-    )
-    (property "Datasheet" "https://www.murata.com/products/productdetail?partno=GRM155R61A475MEAA%23" (at 266.7 114.3 0)
-      (effects (font (size 1.27 1.27) (thickness 0.15)) (justify left bottom) hide)
-    )
-    (property "Manufacturer" "Murata" (at 261.62 114.3 0)
-      (effects (font (size 1.27 1.27) (thickness 0.15)) (justify left bottom) hide)
-    )
-    (property "MPN" "GRM155R61A475MEAAD" (at 264.16 114.3 0)
-      (effects (font (size 1.27 1.27) (thickness 0.15)) (justify left bottom) hide)
-    )
-    (property "Val" "4u7" (at 284.48 98.4312 90)
-      (effects (font (size 1.27 1.27) (thickness 0.15)) (justify left))
-    )
-    (property "License" "Apache-2.0" (at 259.08 114.3 0)
-      (effects (font (size 1.27 1.27) (thickness 0.15)) (justify left bottom) hide)
-    )
-    (property "Author" "Antmicro" (at 256.54 114.3 0)
-      (effects (font (size 1.27 1.27) (thickness 0.15)) (justify left bottom) hide)
-    )
-    (property "Voltage" "" (at 254 114.3 0)
-      (effects (font (size 1.27 1.27)) (justify left bottom) hide)
-    )
-    (property "Dielectric" "" (at 251.46 114.3 0)
-      (effects (font (size 1.27 1.27)) (justify left bottom) hide)
-    )
-    (pin "1")
-    (pin "2")
-    (instances
-      (project "data-center-rdimm-ddr5-tester"
-        (path "/1faa6543-e26a-4449-8bac-ee14b9f19e5f/00000000-0000-0000-0000-000061827943"
-          (reference "C7") (unit 1)
         )
       )
@@
         )
       )
-    )
-  )
-  (symbol (lib_id "antmicroCapacitors0402:C_4u7_0402") (at 281.94 110.49 270) (unit 1)
-    (in_bom yes) (on_board yes) (dnp no) (fields_autoplaced)
-    (property "Reference" "C319" (at 284.48 111.7663 90)
-      (effects (font (size 1.27 1.27)) (justify left))
-    )
-    (property "Value" "C_4u7_0402" (at 271.78 130.81 0)
-      (effects (font (size 1.27 1.27) (thickness 0.15)) (justify left bottom) hide)
-    )
-    (property "Footprint" "antmicro-footprints:C_0402_1005Metric" (at 269.24 130.81 0)
-      (effects (font (size 1.27 1.27) (thickness 0.15)) (justify left bottom) hide)
-    )
-    (property "Datasheet" "https://www.murata.com/products/productdetail?partno=GRM155R61A475MEAA%23" (at 266.7 130.81 0)
-      (effects (font (size 1.27 1.27) (thickness 0.15)) (justify left bottom) hide)
-    )
-    (property "Manufacturer" "Murata" (at 261.62 130.81 0)
-      (effects (font (size 1.27 1.27) (thickness 0.15)) (justify left bottom) hide)
-    )
-    (property "MPN" "GRM155R61A475MEAAD" (at 264.16 130.81 0)
-      (effects (font (size 1.27 1.27) (thickness 0.15)) (justify left bottom) hide)
-    )
-    (property "Val" "4u7" (at 284.48 114.9412 90)
-      (effects (font (size 1.27 1.27) (thickness 0.15)) (justify left))
-    )
-    (property "License" "Apache-2.0" (at 259.08 130.81 0)
-      (effects (font (size 1.27 1.27) (thickness 0.15)) (justify left bottom) hide)
-    )
-    (property "Author" "Antmicro" (at 256.54 130.81 0)
-      (effects (font (size 1.27 1.27) (thickness 0.15)) (justify left bottom) hide)
-    )
-    (property "Voltage" "" (at 254 130.81 0)
-      (effects (font (size 1.27 1.27)) (justify left bottom) hide)
-    )
-    (property "Dielectric" "" (at 251.46 130.81 0)
-      (effects (font (size 1.27 1.27)) (justify left bottom) hide)
-    )
-    (pin "1")
-    (pin "2")
-    (instances
-      (project "data-center-rdimm-ddr5-tester"
-        (path "/1faa6543-e26a-4449-8bac-ee14b9f19e5f/00000000-0000-0000-0000-000061827943"
-          (reference "C319") (unit 1)
-        )
-      )
