File: supply.kicad_sch (KiCad schematic)
At the start: 56 parts, among them J7 BarrelJack_Pin1.3mm_694103107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, J8 JST_SH_1x4_BM04B-SRSS-TB-LF-SN, Q12 SI7613DN-T1-GE3, Q13 SI7613DN-T1-GE3, Q14 BSS138PW, Q15 BSS138PW, Q16 BSS138PW, Q17 BSS138PW, SW4 SW_CVS-08TB, SW5 SW_KMR211NGLFS_SMD, U17 LTC4412IS6, U18 LTC4412IS6, U21 NCP718BSN330T1G, U22 MAX16150A_SOT, U26 MAX812REUS+T, U29 AT24CS01_SOT23, U31 LM3880

Commit message: [#68088] Add heater connector
Parts:
- added C321: C_100n_0402, antmicro-footprints:C_0402_1005Metric, symbol antmicroCapacitors0402:C_100n_0402
- added C323, C326, C327: C_10u_25V_0603, antmicro-footprints:C_0603_1608Metric, symbol antmicroCapacitors0603:C_10u_25V_0603
- added F3: F_1.25A_0603, antmicro-footprints:F_0603_1608Metric, symbol antmicroFuses:F_1.25A_0603
- added J17: JST_SH_1x2_BM02B-SRSS-TB-LF-SN, antmicro-footprints:Conn_JST_SH_1x2_BM02B-SRSS-TB-LF-SN, symbol antmicroWire2BoardConnectors:JST_SH_1x2_BM02B-SRSS-TB-LF-SN
- added Q28: BSS138PW, antmicro-footprints:SC70-3, symbol antmicroTransistorsFETsMOSFETsSingle:BSS138PW
- added Q29: SI7613DN-T1-GE3, antmicro-footprints:Vishay_PowerPAK_1212-8_Single, symbol antmicroTransistorsFETsMOSFETsSingle:SI7613DN-T1-GE3
- added R249, R250: R_47k_0402, antmicro-footprints:R_0402_1005Metric, symbol antmicroResistors0402:R_47k_0402
Connections:
- net GND: now also C321.1, C323.1, C326.1, C327.1, J17.2, J17.MP, Q28.2 (S), R250.1
- net VDC: now also C326.2, C327.2, Q29.1 (S), Q29.2 (S), Q29.3 (S), R249.2
- new net: Q28.3 (D), Q29.4 (G), R249.1
- new net: F3.1, Q29.5 (D)
- new net Heater_PWM: Q28.1 (G), R250.2
- new net heater: C321.2, C323.2, F3.2, J17.1
Other:
- note added: "Heater connector"
- note added: "Max 10W"
- moved on the sheet: C198, J8, Q15, R170
