File: ddr5-sodimm.kicad_sch (KiCad schematic)
At the start: 31 parts, among them J2 Bus_DDR5_SODIMM_Amphenol_1016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, Q10 BSS138PW, Q11 BSS138PW, Q9 BSS138PW, SW3 SW_KMR211NGLFS_SMD

Commit message: [#69629] Fix DNP attributes
Parts:
- C127, R24, R26, R29, R30, R32, R33, R34, R35: DNP DNP -> (none)
