File: hyperram-flash.kicad_sch (KiCad schematic)
At the start: 17 parts, among them U1 IS66WVH16M8DALL-166B1LI, U27 W25Q128JWEIQ

Commit message: Correct company name in project files
Other:
- company: Antmicro Ltd. -> Antmicro
Changed lines of the file:
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@@
 		(date "2024-12-20")
 		(rev "2.1.0")
-		(company "Antmicro Ltd.")
+		(company "Antmicro")
 		(comment 1 "www.antmicro.com")
 		(comment 2 "Antmicro")
