File: pcie-connector.kicad_sch (KiCad schematic)
At the start: 6 parts, among them J10 PCB-Edge_PCIexpress_x8, SW1 CVS-03B

Commit message: Correct company name in project files
Other:
- company: (none) -> Antmicro
Changed lines of the file:
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@@
 		(date "2024-12-20")
 		(rev "2.1.0")
+		(company "Antmicro")
 		(comment 1 "www.antmicro.com")
 		(comment 2 "Antmicro")
