File: dc-dc-aux-mgt.kicad_sch (KiCad schematic)
At the start: 42 parts, among them U19 MPM54304GMN, U25 PAC1720-1, U3 PAC1720-1

Commit message: Correct company name in project files
Other:
- company: (none) -> Antmicro
Changed lines of the file:
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@@
 		(date "2024-12-20")
 		(rev "2.1.0")
+		(company "Antmicro")
 		(comment 1 "www.antmicro.com")
 		(comment 2 "Antmicro")

Commit message: [#97338] Fix malformed DNP properties
Parts:
- TP14, TP15, TP18, TP8: now left out of the parts list
Changed lines of the file:
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@@
 		(unit 1)
 		(exclude_from_sim no)
-		(in_bom yes)
+		(in_bom no)
 		(on_board yes)
 		(dnp no)
@@
 		(unit 1)
 		(exclude_from_sim no)
-		(in_bom yes)
+		(in_bom no)
 		(on_board yes)
 		(dnp no)
@@
 		(unit 1)
 		(exclude_from_sim no)
-		(in_bom yes)
+		(in_bom no)
 		(on_board yes)
 		(dnp no)
@@
 		(unit 1)
 		(exclude_from_sim no)
-		(in_bom yes)
+		(in_bom no)
 		(on_board yes)
 		(dnp no)
