File: dc-dc-vccint.kicad_sch (KiCad schematic)
At the start: 62 parts, among them U36 MP8796B, U4 MP8796B

Commit message: Correct company name in project files
Other:
- company: (none) -> Antmicro
Changed lines of the file:
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@@
 		(date "2024-12-20")
 		(rev "2.1.0")
+		(company "Antmicro")
 		(comment 1 "www.antmicro.com")
 		(comment 2 "Antmicro")

Commit message: [#97338] Fix malformed DNP properties
Parts:
- C313, C314: now in the parts list
- TP10, TP17, TP25, TP26: now left out of the parts list
Changed lines of the file:
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@@
 		(unit 1)
 		(exclude_from_sim no)
-		(in_bom yes)
+		(in_bom no)
 		(on_board yes)
 		(dnp no)
@@
 		(unit 1)
 		(exclude_from_sim no)
-		(in_bom no)
+		(in_bom yes)
 		(on_board yes)
 		(dnp no)
@@
 	)
 	(symbol
+		(lib_name "PWR_FLAG_1")
 		(lib_id "antmicropower:PWR_FLAG")
 		(at 241.3 203.2 0)
@@
 		(unit 1)
 		(exclude_from_sim no)
-		(in_bom yes)
+		(in_bom no)
 		(on_board yes)
 		(dnp no)
@@
 		(unit 1)
 		(exclude_from_sim no)
-		(in_bom yes)
+		(in_bom no)
 		(on_board yes)
 		(dnp no)
@@
 		(unit 1)
 		(exclude_from_sim no)
-		(in_bom no)
+		(in_bom yes)
 		(on_board yes)
 		(dnp no)
@@
 		(unit 1)
 		(exclude_from_sim no)
-		(in_bom yes)
+		(in_bom no)
 		(on_board yes)
 		(dnp no)
