File: debug-ftdi.kicad_sch (KiCad schematic)
At the start: 85 parts, among them J13 U_FL-R-SMT-1, J14 U_FL-R-SMT-1, J15 U_FL-R-SMT-1, J16 U_FL-R-SMT-1, J3 USB-C_GCT_USB4105-GF-A, J9 U_FL-R-SMT-1, Q20 BSS84AKW, U13 TXU0304BQAR, U16 TXS0102DQER, U32 TXS0102DQER, U5 NCP718BSN330T1G, U6 FT4232H_VQFN, U7 TXU0304BQAR, U8 TPD4E05U06QDQARQ1, U9 SN74HC595B, Y1 Resonator_12MHz_ABM8G

Commit message: Correct company name in project files
Other:
- company: Antmicro Ltd. -> Antmicro
Changed lines of the file:
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@@
 		(date "2024-12-20")
 		(rev "2.1.0")
-		(company "Antmicro Ltd.")
+		(company "Antmicro")
 		(comment 1 "www.antmicro.com")
 		(comment 2 "Antmicro")

Commit message: [#97338] Fix malformed DNP properties
Parts:
- TP1, TP22: now left out of the parts list
Changed lines of the file:
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@@
 		(unit 1)
 		(exclude_from_sim no)
-		(in_bom yes)
+		(in_bom no)
 		(on_board yes)
 		(dnp no)
@@
 		(unit 1)
 		(exclude_from_sim no)
-		(in_bom yes)
+		(in_bom no)
 		(on_board yes)
 		(dnp no)
